Commit message: update

File: install/arduinobot_description/share/arduinobot_description/urdf/arduinobot_ros2_control.xacro (robot description, xacro)
@@ -41,8 +41,8 @@
             <state_interface name="position"/>
         </joint>
-        <joint name="joint_5">
+        <!-- <joint name="joint_5">
             <param name="mimic">joint_4</param>
             <param name="multiplier">-1</param>
-        </joint>
+        </joint> -->
     </ros2_control>
 </robot>
